File: rev1_savi/rev1_savi.kicad_sch (KiCad schematic)
At the start: 0 parts

Commit message: Add files via upload
Schematic for IMU, Lidar, Pi
Parts:
- added J1: Raspberry_Pi_4, symbol Connector:Raspberry_Pi_4
- added R1, R2: 4.7k, symbol Device:R
- added U2: ICM-20948, Sensor_Motion:InvenSense_QFN-24_3x3mm_P0.4mm, symbol Sensor_Motion:ICM-20948
- added U4: TFmini_S Lidar, symbol sensors:TFmini_S
Connections:
- new net: J1.1 (3V3), J1.17 (3V3)
- new net +3.3V: R1.2, R2.2, U2.13 (VDD), U2.22 (~{CS}), U2.8 (VDDIO)
- new net GND: J1.14 (GND), J1.20 (GND), J1.25 (GND), J1.30 (GND), J1.34 (GND), J1.39 (GND), J1.6 (GND), J1.9 (GND), U2.18 (GND), U2.20 (GND), U2.9 (SDO/AD0), U4.1 (GND)
- new net I2C_SCL: J1.5 (SCL_I2C1/GPIO03), R2.1, U2.23 (SCL/SCLK), U4.4 (SCL)
- new net I2C_SDA: J1.3 (SDA_I2C1/GPIO02), R1.1, U2.24 (SDA/SDI), U4.3 (SDA)
- new net Pi_5V: J1.2 (5V), J1.4 (5V), U4.2 (+5V)
Other:
- title: (none) -> SAVI I2C Sensor Bus (Pi + LiDAR + BNO055)

Commit message: Update rev1_savi.kicad_sch: changed IMU name
Other:
- title: SAVI I2C Sensor Bus (Pi + LiDAR + BNO055) -> SAVI I2C Sensor Bus (Pi + LiDAR + ICM-20948)
Changed lines of the file:
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@@
 	(paper "A4")
 	(title_block
-		(title "SAVI I2C Sensor Bus (Pi + LiDAR + BNO055)")
+		(title "SAVI I2C Sensor Bus (Pi + LiDAR + ICM-20948)")
 	)
 	(junction

Commit message: Add files via upload
Parts:
- removed U2: ICM-20948, Sensor_Motion:InvenSense_QFN-24_3x3mm_P0.4mm, symbol Sensor_Motion:ICM-20948
- added U1: BNO055_IC2, symbol sensors:BNO055_IC2
Connections:
- net +3.3V: now also U1.11 (nRESET), U1.28 (VDDIO), U1.3 (VDD), U1.4 (nBOOT_LOAD_PIN)
- net GND: now also U1.10 (GNDIO), U1.15 (GNDIO), U1.16 (GNDIO), U1.2 (GND), U1.25 (GNDIO), U1.5 (PS1), U1.6 (PS0)
- net I2C_SCL: now also U1.19 (SCL)
- net I2C_SDA: now also U1.20 (SDA)
Other:
- title: SAVI I2C Sensor Bus (Pi + LiDAR + ICM-20948) -> SAVI I2C Sensor Bus (Pi + LiDAR + BNO055)
